File: Schematics/sample_application.sch (EAGLE design)
At the start: 33 parts, among them K1 ZF112, K2 ZF112, K3 ZF112, K4 ZF112, T1 IRLZ44Z, T2 IRLZ44Z, T3 IRLZ44Z, T4 IRLZ44Z

Commit message: Added optional pull-up resistor and note to schematics
Parts:
- added R1: (no value), resistor:R-EU_0204/5
Connections:
- net N$8: now also R1.1
- net VCC: now also R1.2
Other:
- note added: "Add 470R <= R1 <= 1K for improved EMC immunity, if wires to switch cannot be kept short"
Changed lines of the file:
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@@
 <part name="SUPPLY5" library="supply2" library_urn="urn:adsk.eagle:library:372" deviceset="VCC" device="" value="N"/>
 <part name="C1" library="docu-dummy" library_urn="urn:adsk.eagle:library:215" deviceset="ELKO" device=""/>
+<part name="R1" library="resistor" library_urn="urn:adsk.eagle:library:348" deviceset="R-EU_" device="0204/5" package3d_urn="urn:adsk.eagle:package:25955/1"/>
+<part name="P+6" library="supply1" library_urn="urn:adsk.eagle:library:371" deviceset="VCC" device=""/>
 </parts>
 <sheets>
@@
 </text>
 <wire x1="-12.7" y1="30.48" x2="71.12" y2="30.48" width="0.1524" layer="104"/>
+<text x="88.9" y="-15.24" size="2.54" layer="104">Add 470R &lt;= R1 &lt;= 1K for improved
+EMC immunity, if wires to switch cannot
+be kept short</text>
 </plain>
 <instances>
@@
 <instance part="SUPPLY5" gate="G$1" x="-2.54" y="-48.26" rot="R90"/>
 <instance part="C1" gate="G$1" x="149.86" y="30.48"/>
+<instance part="R1" gate="G$1" x="116.84" y="111.76"/>
+<instance part="P+6" gate="VCC" x="124.46" y="111.76" rot="R270"/>
 </instances>
 <busses>
@@
 <pinref part="B1" gate="G$1" pin="D2"/>
 <wire x1="111.76" y1="73.66" x2="119.38" y2="73.66" width="0.1524" layer="91"/>
+<pinref part="R1" gate="G$1" pin="1"/>
+<junction x="111.76" y="111.76"/>
 </segment>
 </net>
@@
 <junction x="53.34" y="-48.26"/>
 </segment>
-</net>
+<segment>
+<pinref part="R1" gate="G$1" pin="2"/>
+<pinref part="P+6" gate="VCC" pin="VCC"/>
+</segment>
+</net>
