File: Schematics/wiring.sch (EAGLE design)
At the start: 17 parts

Commit message: Added optional pull-up resistor and note to schematics
Parts:
- added R1: (no value), resistor:R-EU_0204/5
Connections:
- net N$8: now also R1.1
- net VCC: now also R1.2
Other:
- note added: "Add 470R <= R1 <= 1K for improved EMC immunity, if wires to switch cannot be kept short"
Changed lines of the file:
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@@
 <part name="GND12" library="supply1" library_urn="urn:adsk.eagle:library:371" deviceset="GND" device=""/>
 <part name="P+1" library="supply1" library_urn="urn:adsk.eagle:library:371" deviceset="VCC" device=""/>
+<part name="R1" library="resistor" library_urn="urn:adsk.eagle:library:348" deviceset="R-EU_" device="0204/5" package3d_urn="urn:adsk.eagle:package:25955/1"/>
+<part name="P+2" library="supply1" library_urn="urn:adsk.eagle:library:371" deviceset="VCC" device=""/>
 </parts>
 <sheets>
@@
 <text x="-20.32" y="7.62" size="2.54" layer="104">HM-LC-Sw4-Ba-PCB and Arduino MUST share a common ground
 HM-LC-Sw4-Ba-PCB and Arduino MAY share VCC/UB+</text>
+<text x="114.3" y="91.44" size="2.54" layer="104">Add 470R &lt;= R1 &lt;= 1K
+for improved EMC immunity,
+if wires to switch cannot be
+kept short</text>
 </plain>
 <instances>
@@
 <instance part="GND12" gate="1" x="91.44" y="10.16" rot="R270"/>
 <instance part="P+1" gate="VCC" x="147.32" y="35.56" rot="R270"/>
+<instance part="R1" gate="G$1" x="116.84" y="111.76"/>
+<instance part="P+2" gate="VCC" x="124.46" y="111.76" rot="R270"/>
 </instances>
 <busses>
@@
 <pinref part="B1" gate="G$1" pin="D2"/>
 <wire x1="111.76" y1="73.66" x2="119.38" y2="73.66" width="0.1524" layer="91"/>
+<pinref part="R1" gate="G$1" pin="1"/>
+<junction x="111.76" y="111.76"/>
 </segment>
 </net>
@@
 <pinref part="P+1" gate="VCC" pin="VCC"/>
 </segment>
-</net>
+<segment>
+<pinref part="R1" gate="G$1" pin="2"/>
+<pinref part="P+2" gate="VCC" pin="VCC"/>
+</segment>
+</net>
